File: PCB/OpenTag/OpenTag.kicad_sch (KiCad schematic)
At the start: 0 parts

Commit message: Update PCB
Parts:
- added ESP32-1, ESP32-2: Conn_01x17, Connector_PinSocket_2.54mm:PinSocket_1x17_P2.54mm_Vertical, symbol Connector_Generic:Conn_01x17
- added H1, H2, H3, H4: MountingHole, MountingHole:MountingHole_3.2mm_M3, symbol Mechanical:MountingHole
- added J1: Conn_01x02, Connector_JST:JST_EH_B2B-EH-A_1x02_P2.50mm_Vertical, symbol Connector_Generic:Conn_01x02
Connections:
- new net 3V: ESP32-1.1 (Pin_1)
- new net 5V: J1.1 (Pin_1)
- new net GND: ESP32-1.12 (Pin_12), ESP32-2.17 (Pin_17), J1.2 (Pin_2)
